File: pcb/DreamPicoPortSchem.sch (EAGLE design)
At the start: 57 parts, among them J1 FFC3B07-20-T

Commit message: 177: Uploaded Rev 1.0 board files
Parts:
- removed R29, R30, R31, R32, R33, R34, R35, R36: NP, Jumper Pad:R_CHIP-0402(1005-METRIC)
- added JP10, JP11, JP12, JP5, JP6, JP7, JP8, JP9: JUMPER-SMT_2_NO_NO-SILK, SparkFun-Jumpers:JUMPER-SMT_2_NO_NO-SILK
- added R8: 120, Tinkercad:RESISTOR__CHIP-0603(1608-METRIC)
- renumbered C5 to C1
Connections:
- net +3.3V: now also R8.1
- net N$11: now also JP10.1; no longer R34.2
- net N$13: now also JP8.2; no longer R32.1
- net N$15: now also JP7.2; no longer R31.1
- net N$17: now also R8.2
- net N$18: now also JP8.1; no longer R32.2
- net N$19: now also JP7.1; no longer R31.2
- net N$21: now also JP5.2; no longer R29.1
- net N$22: now also JP9.1; no longer R33.2
- net N$25: now also JP10.2; no longer R34.1
- net N$26: now also JP9.2; no longer R33.1
- net N$29: now also JP12.1; no longer R36.2
- net N$3: now also JP6.2; no longer R30.1
- net N$30: now also JP11.1; no longer R35.2
- net N$36: now also JP12.2; no longer R36.1
- net N$37: now also JP11.2; no longer R35.1
- net N$6: now also JP5.1; no longer R29.2
- net N$7: now also JP6.1; no longer R30.2

Commit message: 177: Changed R[A-D]1 and R[A-D]2 resistors to 1206 size
Parts:
- RA1, RA2, RB1, RB2, RC1, RC2, RD1, RD2: device Tinkercad:RESISTOR__CHIP-0603(1608-METRIC) -> Resistor:R_CHIP-1206(3216-METRIC)
