File: pcb/DreamPicoPortSchem.sch (EAGLE design)
At the start: 57 parts, among them J1 FFC3B07-20-T

Commit message: 177: Uploaded Rev 1.0 board files (#180)
* 177: Uploaded Rev 1.0 board files

* 177: Changed R[A-D]1 and R[A-D]2 resistors to 1206 size

* 177: Mask vias on PCB

* 177: Added board examples

---------

Co-authored-by: James Smith <{ID}+{username}@users.noreply.github.com>
Parts:
- removed R29, R30, R31, R32, R33, R34, R35, R36: NP, Jumper Pad:R_CHIP-0402(1005-METRIC)
- added JP10, JP11, JP12, JP5, JP6, JP7, JP8, JP9: JUMPER-SMT_2_NO_NO-SILK, SparkFun-Jumpers:JUMPER-SMT_2_NO_NO-SILK
- added R8: 120, Tinkercad:RESISTOR__CHIP-0603(1608-METRIC)
- RA1, RA2, RB1, RB2, RC1, RC2, RD1, RD2: device Tinkercad:RESISTOR__CHIP-0603(1608-METRIC) -> Resistor:R_CHIP-1206(3216-METRIC)
- renumbered C5 to C1
Connections:
- net +3.3V: now also R8.1
- net N$11: now also JP10.1; no longer R34.2
- net N$13: now also JP8.2; no longer R32.1
- net N$15: now also JP7.2; no longer R31.1
- net N$17: now also R8.2
- net N$18: now also JP8.1; no longer R32.2
- net N$19: now also JP7.1; no longer R31.2
- net N$21: now also JP5.2; no longer R29.1
- net N$22: now also JP9.1; no longer R33.2
- net N$25: now also JP10.2; no longer R34.1
- net N$26: now also JP9.2; no longer R33.1
- net N$29: now also JP12.1; no longer R36.2
- net N$3: now also JP6.2; no longer R30.1
- net N$30: now also JP11.1; no longer R35.2
- net N$36: now also JP12.2; no longer R36.1
- net N$37: now also JP11.2; no longer R35.1
- net N$6: now also JP5.1; no longer R29.2
- net N$7: now also JP6.1; no longer R30.2

Commit message: Updated 5V to VBUS on PCB
Parts:
- added JP13: JUMPER-SMT_2_NO_NO-SILK, SparkFun-Jumpers:JUMPER-SMT_2_NO_NO-SILK
Connections:
- new net N$24: JP13.2, U1.VSYS
- net +5V: now also JP13.1, U1.VBUS; no longer U1.VSYS
Changed lines of the file:
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@@
 <part name="R8" library="Tinkercad" library_urn="urn:adsk.eagle:library:30890021" deviceset="RESISTOR" device="_CHIP-0603(1608-METRIC)" package3d_urn="urn:adsk.eagle:package:16378565/5" technology="_" value="120"/>
 <part name="SUPPLY22" library="Tutorial - Fusion 360" library_urn="urn:adsk.eagle:library:16997205" deviceset="VCC-BAR" device="" value="+3.3V"/>
+<part name="JP13" library="SparkFun-Jumpers" deviceset="JUMPER-SMT_2_NO" device="_NO-SILK" package3d_urn="urn:adsk.eagle:package:39277/1"/>
 </parts>
 <sheets>
@@
 <attribute name="VALUE" x="320.167" y="-3.175" size="1.778" layer="96" align="bottom-center"/>
 </instance>
-<instance part="SUPPLY21" gate="G$1" x="83.82" y="88.9" smashed="yes">
-<attribute name="VALUE" x="83.82" y="89.408" size="1.778" layer="96" align="bottom-center"/>
+<instance part="SUPPLY21" gate="G$1" x="71.12" y="114.3" smashed="yes">
+<attribute name="VALUE" x="71.12" y="114.808" size="1.778" layer="96" align="bottom-center"/>
 </instance>
 <instance part="SUPPLY23" gate="G$1" x="96.52" y="10.16" smashed="yes">
@@
 <instance part="SUPPLY22" gate="G$1" x="114.3" y="-30.48" smashed="yes">
 <attribute name="VALUE" x="114.3" y="-29.972" size="1.778" layer="96" align="bottom-center"/>
+</instance>
+<instance part="JP13" gate="G$1" x="78.74" y="104.14" smashed="yes">
+<attribute name="NAME" x="78.74" y="106.934" size="1.778" layer="95" font="vector" align="center"/>
+<attribute name="VALUE" x="78.74" y="101.346" size="1.778" layer="96" font="vector" align="center"/>
 </instance>
 </instances>
@@
 </segment>
 <segment>
-<wire x1="71.12" y1="81.28" x2="83.82" y2="81.28" width="0.1524" layer="91"/>
-<wire x1="83.82" y1="81.28" x2="83.82" y2="86.36" width="0.1524" layer="91"/>
+<pinref part="JP13" gate="G$1" pin="1"/>
+<wire x1="71.12" y1="83.82" x2="71.12" y2="104.14" width="0.1524" layer="91"/>
+<wire x1="71.12" y1="104.14" x2="73.66" y2="104.14" width="0.1524" layer="91"/>
+<pinref part="U1" gate="G$1" pin="VBUS"/>
+<wire x1="71.12" y1="104.14" x2="71.12" y2="111.76" width="0.1524" layer="91"/>
+<junction x="71.12" y="104.14"/>
 <pinref part="SUPPLY21" gate="G$1" pin="VCC"/>
-<wire x1="83.82" y1="81.28" x2="96.52" y2="81.28" width="0.1524" layer="91"/>
-<junction x="83.82" y="81.28"/>
-<pinref part="U1" gate="G$1" pin="VSYS"/>
+<wire x1="71.12" y1="111.76" x2="71.12" y2="109.22" width="0.1524" layer="91"/>
+<wire x1="71.12" y1="109.22" x2="96.52" y2="109.22" width="0.1524" layer="91"/>
+<junction x="71.12" y="111.76"/>
+<wire x1="96.52" y1="109.22" x2="96.52" y2="81.28" width="0.1524" layer="91"/>
 <pinref part="C1" gate="A" pin="1"/>
 </segment>
@@
 </segment>
 </net>
+<net name="N$24" class="0">
+<segment>
+<pinref part="JP13" gate="G$1" pin="2"/>
+<wire x1="83.82" y1="104.14" x2="83.82" y2="81.28" width="0.1524" layer="91"/>
+<wire x1="83.82" y1="81.28" x2="71.12" y2="81.28" width="0.1524" layer="91"/>
+<pinref part="U1" gate="G$1" pin="VSYS"/>
+</segment>
+</net>
